File: CESP.sch (KiCad schematic (older format))
At the start: 5 parts

Commit message: Soldering practice board slapped together
Parts:
- removed U?: LTC1594CS, TSSOP14, symbol LTC1594CS
- removed U?: TL074, TSSOP14, symbol TL074
- removed U? (x3): TL074, symbol TL074
- added C1, C2: C 2.5, symbol C
- added C3, C4: C 5, symbol C
- added IC1: SOT23-6, SOT23-6, symbol ATTINY9-TS
- added IC2: TSSOP20, TSSOP20, symbol ATTINY40-X
- added IC3: SOIC16, SO20, symbol ATTINY40-SU
- added IC4: TQFP64, TQFP100, symbol ATMEGA1280-A
- added Q1, Q8, Q9: SOT23, symbol MOSFET_N
- added Q2: D2PAK, symbol MOSFET_N
- added Q3, Q4: TO92, symbol MOSFET_N
- added Q5, Q6: TO220, symbol MOSFET_N
- added Q7: TO247, symbol MOSFET_N
- added R1, R2, R3, R4: 0402, symbol R
- added R10, R11, R12, R9: 0805, symbol R
- added R13, R14: 1206, symbol R
- added R15: 1210, symbol R
- added R16: 2512, symbol R
- added R17, R18: R VERT, symbol R
- added R19: R HOR, symbol R
- added R20: R HORI, symbol R
- added R5, R6, R7, R8: 0603, symbol R
Connections:
- net labels added: GND
- wire segments 0 -> 15
Other:
- note removed: "NOTE: THIS IS JUST A TEST BOARD\nREMOVE ALL COMPONENTS AND CREATE YOUR OWN\nINCLUDE SCHEMATIC HOOKUPS/NETLIST"
